Commit message: new spectrometer design working in rviz

File: install/mycobot_description/share/mycobot_description/urdf/mycobot_280_urdf.xacro (robot description, xacro)
@@ -176,4 +176,42 @@
 		</inertial>
   </link>
+   <link name="holder">
+  <visual>
+    <origin xyz="0 0 0" rpy="0 0 0"/>
+    <geometry>
+      <mesh filename="file://$(find mycobot_description)/meshes/mycobot_280/holder.stl"/>
+    </geometry>
+  </visual>
+  <collision>
+    <origin xyz="0 0 0" rpy="0 0 0"/>
+    <geometry>
+      <mesh filename="file://$(find mycobot_description)/meshes/mycobot_280/holder.stl"/>
+    </geometry>
+  </collision>
+   <inertial>
+    <origin xyz="1.257105390531987e-13 1.2571147787950272e-13 2.8451187525301305e-14" rpy="0 0 0"/>
+    <mass value="5.2360263698612974e-11"/>
+    <inertia ixx="0.0" iyy="0.0" izz="0.0" ixy="0.0" iyz="0.0" ixz="0.0"/>
+  </inertial>
+</link>
+<link name="spectrometer">
+  <visual>
+    <origin xyz="-1.3e-05 -0.0 -1e-05" rpy="0 0 0"/>
+    <geometry>
+      <mesh filename="file://$(find mycobot_description)/meshes/mycobot_280/spectrometer.stl"/>
+    </geometry>
+  </visual>
+  <collision>
+    <origin xyz="-1.3e-05 -0.0 -1e-05" rpy="0 0 0"/>
+    <geometry>
+     <mesh filename="file://$(find mycobot_description)/meshes/mycobot_280/spectrometer.stl"/>
+    </geometry>
+  </collision>
+   <inertial>
+    <origin xyz="4.249999739073161e-06 1.024970783172406e-14 -2.4999998975029586e-07" rpy="0 0 0"/>
+    <mass value="1.893181328918444e-11"/>
+    <inertia ixx="0.0" iyy="0.0" izz="0.0" ixy="-0.0" iyz="0.0" ixz="-0.0"/>
+  </inertial>
+</link>
 <!-- ********** JOINTS ********** -->
 <!-- Attach the robot base to the world frame with no initial offset or rotation. -->
@@ -234,3 +272,13 @@
         <dynamics damping="0.01" friction="0.005"/>
 	</joint>
+  <joint name="robot to holder" type="fixed">
+  <origin xyz="1.3e-05 0.0 1e-05" rpy="0 0 0"/>
+  <parent link="link5_flange"/>
+  <child link="holder"/>
+</joint>
+<joint name="Rigid 1" type="fixed">
+  <origin xyz="0.0 0.0 0.0" rpy="0 0 0"/>
+  <parent link="holder"/>
+  <child link="spectrometer"/>
+</joint>
 </robot>

Commit message: New spectrometer working moveit and gazebo

File: install/mycobot_description/share/mycobot_description/urdf/mycobot_280_urdf.xacro (robot description, xacro)
@@ -176,41 +176,43 @@
 		</inertial>
   </link>
-   <link name="holder">
+  <link name="holder">
+  <inertial>
+    <origin xyz="9.542063908505497e-10 4.713475046347886e-13 0.051986133375594434" rpy="0 0 0"/>
+    <mass value="2.1138978819045212e-10"/>
+    <inertia ixx="0.0" iyy="0.0" izz="0.0" ixy="0.0" iyz="0.0" ixz="0.0"/>
+  </inertial>
   <visual>
     <origin xyz="0 0 0" rpy="0 0 0"/>
     <geometry>
-      <mesh filename="file://$(find mycobot_description)/meshes/mycobot_280/holder.stl"/>
-    </geometry>
+     <mesh filename="file://$(find mycobot_description)/meshes/mycobot_280/holder.stl"/>
+    </geometry>
+    <material name="silver"/>
   </visual>
   <collision>
     <origin xyz="0 0 0" rpy="0 0 0"/>
     <geometry>
-      <mesh filename="file://$(find mycobot_description)/meshes/mycobot_280/holder.stl"/>
+     <mesh filename="file://$(find mycobot_description)/meshes/mycobot_280/holder.stl"/>
     </geometry>
   </collision>
-   <inertial>
-    <origin xyz="1.257105390531987e-13 1.2571147787950272e-13 2.8451187525301305e-14" rpy="0 0 0"/>
-    <mass value="5.2360263698612974e-11"/>
-    <inertia ixx="0.0" iyy="0.0" izz="0.0" ixy="0.0" iyz="0.0" ixz="0.0"/>
-  </inertial>
 </link>
 <link name="spectrometer">
+  <inertial>
+    <origin xyz="9.614911284733845e-13 -7.7769165452601e-15 -0.07613934716557663" rpy="0 0 0"/>
+    <mass value="1.4364425990347802e-11"/>
+    <inertia ixx="0.0" iyy="0.0" izz="0.0" ixy="-0.0" iyz="0.0" ixz="-0.0"/>
+  </inertial>
   <visual>
-    <origin xyz="-1.3e-05 -0.0 -1e-05" rpy="0 0 0"/>
-    <geometry>
-      <mesh filename="file://$(find mycobot_description)/meshes/mycobot_280/spectrometer.stl"/>
-    </geometry>
+    <origin xyz="-0.0 -0.0 -0.052052" rpy="0 0 0"/>
+    <geometry>
+     <mesh filename="file://$(find mycobot_description)/meshes/mycobot_280/spectrometer.stl"/>
+    </geometry>
+    <material name="silver"/>
   </visual>
   <collision>
-    <origin xyz="-1.3e-05 -0.0 -1e-05" rpy="0 0 0"/>
+    <origin xyz="-0.0 -0.0 -0.052052" rpy="0 0 0"/>
     <geometry>
      <mesh filename="file://$(find mycobot_description)/meshes/mycobot_280/spectrometer.stl"/>
     </geometry>
   </collision>
-   <inertial>
-    <origin xyz="4.249999739073161e-06 1.024970783172406e-14 -2.4999998975029586e-07" rpy="0 0 0"/>
-    <mass value="1.893181328918444e-11"/>
-    <inertia ixx="0.0" iyy="0.0" izz="0.0" ixy="-0.0" iyz="0.0" ixz="-0.0"/>
-  </inertial>
 </link>
 <!-- ********** JOINTS ********** -->
@@ -272,10 +274,10 @@
         <dynamics damping="0.01" friction="0.005"/>
 	</joint>
-  <joint name="robot to holder" type="fixed">
+  <joint name="robot_to_holder" type="fixed">
   <origin xyz="1.3e-05 0.0 1e-05" rpy="0 0 0"/>
   <parent link="link5_flange"/>
   <child link="holder"/>
 </joint>
-<joint name="Rigid 1" type="fixed">
+<joint name="holder_to_spectrometer" type="fixed">
   <origin xyz="0.0 0.0 0.0" rpy="0 0 0"/>
   <parent link="holder"/>

File: install/mycobot_gazebo/share/mycobot_gazebo/urdf/mycobot_280_classic_gazebo.urdf.xacro (robot description, xacro)
@@ -185,4 +185,44 @@
 		</inertial>
   </link>
+  <link name="holder">
+  <inertial>
+    <origin xyz="9.542063908505497e-10 4.713475046347886e-13 0.051986133375594434" rpy="0 0 0"/>
+    <mass value="2.1138978819045212e-10"/>
+    <inertia ixx="0.0" iyy="0.0" izz="0.0" ixy="0.0" iyz="0.0" ixz="0.0"/>
+  </inertial>
+  <visual>
+    <origin xyz="0 0 0" rpy="0 0 0"/>
+    <geometry>
+     <mesh filename="file://$(find mycobot_description)/meshes/mycobot_280/holder.stl"/>
+    </geometry>
+    <material name="silver"/>
+  </visual>
+  <collision>
+    <origin xyz="0 0 0" rpy="0 0 0"/>
+    <geometry>
+     <mesh filename="file://$(find mycobot_description)/meshes/mycobot_280/holder.stl"/>
+    </geometry>
+  </collision>
+</link>
+<link name="spectrometer">
+  <inertial>
+    <origin xyz="9.614911284733845e-13 -7.7769165452601e-15 -0.07613934716557663" rpy="0 0 0"/>
+    <mass value="1.4364425990347802e-11"/>
+    <inertia ixx="0.0" iyy="0.0" izz="0.0" ixy="-0.0" iyz="0.0" ixz="-0.0"/>
+  </inertial>
+  <visual>
+    <origin xyz="-0.0 -0.0 -0.052052" rpy="0 0 0"/>
+    <geometry>
+     <mesh filename="file://$(find mycobot_description)/meshes/mycobot_280/spectrometer.stl"/>
+    </geometry>
+    <material name="silver"/>
+  </visual>
+  <collision>
+    <origin xyz="-0.0 -0.0 -0.052052" rpy="0 0 0"/>
+    <geometry>
+     <mesh filename="file://$(find mycobot_description)/meshes/mycobot_280/spectrometer.stl"/>
+    </geometry>
+  </collision>
+</link>
   <gazebo reference="base_link">
         <material>Gazebo/Green</material>
@@ -264,4 +304,14 @@
         <dynamics damping="0.01" friction="0.005"/>
 	</joint>
+  <joint name="robot_to_holder" type="fixed">
+  <origin xyz="1.3e-05 0.0 1e-05" rpy="0 0 0"/>
+  <parent link="link5_flange"/>
+  <child link="holder"/>
+</joint>
+<joint name="holder_to_spectrometer" type="fixed">
+  <origin xyz="0.0 0.0 0.0" rpy="0 0 0"/>
+  <parent link="holder"/>
+  <child link="spectrometer"/>
+</joint>
  <!-- ********** PLUGINS ********** -->
     <!-- Publishes joint state information for the model which the robot_state_publisher uses to broadcast to
@@ -276,4 +326,6 @@
             <joint_name>link4_to_link5</joint_name>
             <joint_name>link5_to_link5_flange</joint_name>
+            <joint_name>robot_to_holder</joint_name>
+            <joint_name>holder_to_spectrometer</joint_name>
         </plugin>
     </gazebo>

File: install/mycobot_gazebo/share/mycobot_gazebo/urdf/ros2_control/classic_gazebo/mycobot_280.urdf.xacro (robot description, xacro)
@@ -196,4 +196,44 @@
 		</inertial>
   </link>
+    <link name="holder">
+  <inertial>
+    <origin xyz="9.542063908505497e-10 4.713475046347886e-13 0.051986133375594434" rpy="0 0 0"/>
+    <mass value="2.1138978819045212e-10"/>
+    <inertia ixx="0.0" iyy="0.0" izz="0.0" ixy="0.0" iyz="0.0" ixz="0.0"/>
+  </inertial>
+  <visual>
+    <origin xyz="0 0 0" rpy="0 0 0"/>
+    <geometry>
+     <mesh filename="file://$(find mycobot_description)/meshes/mycobot_280/holder.stl"/>
+    </geometry>
+    <material name="silver"/>
+  </visual>
+  <collision>
+    <origin xyz="0 0 0" rpy="0 0 0"/>
+    <geometry>
+     <mesh filename="file://$(find mycobot_description)/meshes/mycobot_280/holder.stl"/>
+    </geometry>
+  </collision>
+</link>
+<link name="spectrometer">
+  <inertial>
+    <origin xyz="9.614911284733845e-13 -7.7769165452601e-15 -0.07613934716557663" rpy="0 0 0"/>
+    <mass value="1.4364425990347802e-11"/>
+    <inertia ixx="0.0" iyy="0.0" izz="0.0" ixy="-0.0" iyz="0.0" ixz="-0.0"/>
+  </inertial>
+  <visual>
+    <origin xyz="-0.0 -0.0 -0.052052" rpy="0 0 0"/>
+    <geometry>
+     <mesh filename="file://$(find mycobot_description)/meshes/mycobot_280/spectrometer.stl"/>
+    </geometry>
+    <material name="silver"/>
+  </visual>
+  <collision>
+    <origin xyz="-0.0 -0.0 -0.052052" rpy="0 0 0"/>
+    <geometry>
+     <mesh filename="file://$(find mycobot_description)/meshes/mycobot_280/spectrometer.stl"/>
+    </geometry>
+  </collision>
+</link>
   <gazebo reference="base_link">
         <material>Gazebo/Green</material>
@@ -273,4 +313,14 @@
         <dynamics damping="0.01" friction="0.005"/>
 	</joint>
+  <joint name="robot_to_holder" type="fixed">
+  <origin xyz="1.3e-05 0.0 1e-05" rpy="0 0 0"/>
+  <parent link="link5_flange"/>
+  <child link="holder"/>
+</joint>
+<joint name="holder_to_spectrometer" type="fixed">
+  <origin xyz="0.0 0.0 0.0" rpy="0 0 0"/>
+  <parent link="holder"/>
+  <child link="spectrometer"/>
+</joint>
     <xacro:default_transmission joint_name="base_link_to_link1"/>
     <xacro:default_transmission joint_name="link1_to_link2"/>
