Commit message: giving robot poses working while listening to topic

File: src/mycobot_ros2/mycobot_description/urdf/mycobot_280_urdf.xacro (robot description, xacro)
@@ -1,5 +1,25 @@
-<?xml version="1.0"?>
-<robot  xmlns:xacro="http://www.ros.org/wiki/xacro" name="firefighter" >
+<?xml version="1.0" ?>
+<robot xmlns:xacro="http://wiki.ros.org/xacro" name="mycobot_280">
+    <xacro:include filename="$(find mycobot_gazebo)/urdf/ros2_control/classic_gazebo/mycobot_280_classic_gazebo.xacro"/>
+    <xacro:include filename="$(find mycobot_gazebo)/urdf/ros2_control/classic_gazebo/mycobot_280_ros2_control.xacro"/>
+    <xacro:macro name="default_transmission" params="joint_name">
+        <transmission name="transmission_${joint_name}">
+            <plugin>transmission_interface/SimpleTransmission</plugin>
+            <actuator name="actuator_${joint_name}" role="actuator_${joint_name}"/>
+            <joint name="${joint_name}" role="${joint_name}">
+                <mechanical_reduction>1.0</mechanical_reduction>
+            </joint>
+        </transmission>
+    </xacro:macro>
 <xacro:property name="width" value=".2" />
+  <material name="white">
+        <color rgba="1 1 1 1"/>
+    </material>
+    <material name="orange">
+        <color rgba="1 0.3 0.1 1"/>
+    </material>
+    <material name="blue">
+        <color rgba="0.2 0.2 1 1"/>
+    </material>
 <material name="silver">
   <color rgba="0.75 0.75 0.75 1.0"/>
@@ -12,5 +32,5 @@
 	<xacro:property name="velocity" value="2.792527"/>
 	<!-- ********** LINKS ********** -->
-  <link name="joint1">
+  <link name="base_link">
     <visual>
       <geometry>
@@ -176,5 +196,5 @@
 		</inertial>
   </link>
-  <link name="holder">
+    <link name="holder">
   <inertial>
     <origin xyz="9.542063908505497e-10 4.713475046347886e-13 0.051986133375594434" rpy="0 0 0"/>
@@ -216,4 +236,25 @@
   </collision>
 </link>
+  <gazebo reference="base_link">
+        <material>Gazebo/Green</material>
+    </gazebo>
+    <gazebo reference="link1">
+        <material>Gazebo/Blue</material>
+    </gazebo>
+    <gazebo reference="link2">
+        <material>Gazebo/Orange</material>
+    </gazebo>
+<gazebo reference="link3">
+        <material>Gazebo/Green</material>
+    </gazebo>
+    <gazebo reference="link4">
+        <material>Gazebo/Blue</material>
+    </gazebo>
+    <gazebo reference="link5">
+        <material>Gazebo/Orange</material>
+    </gazebo>
+      <gazebo reference="link5_flange">
+        <material>Gazebo/Green</material>
+    </gazebo>
 <!-- ********** JOINTS ********** -->
 <!-- Attach the robot base to the world frame with no initial offset or rotation. -->
@@ -221,18 +262,16 @@
 	<joint name="virtual_joint" type="fixed">
 		<parent link="world"/>
-		<child link="joint1"/>
-		<origin xyz= "0 0 0" rpy = "0 0 0"/>
-	</joint>
-	<!-- Define the joint name and its type as "fixed". A fixed joint
-	means the two connected links cannot move relative to each other. -->
-		<joint name="joint1" type="revolute">
+		<child link="base_link"/>
+		<origin xyz= "0 0 -0.05" rpy = "0 0 0"/>
+	</joint>
+<joint name="base_link_to_link1" type="revolute">
 		<axis xyz="0 0 1"/>
 		<limit effort = "${effort}" lower = "-2.879793" upper = "2.879793" velocity = "${velocity}"/>
-		<parent link="joint1"/>
+		<parent link="base_link"/>
 		<child link="link1"/>
 	    <origin xyz= "0 0 0.13156" rpy = "0 0 ${pi/2}"/>
         <dynamics damping="0.05" friction="0.05"/>
 	</joint>
-	<joint name="joint2" type="revolute">
+	<joint name="link1_to_link2" type="revolute">
 		<axis xyz="0 0 1"/>
 		<limit effort = "${effort}" lower = "-2.879793" upper = "2.879793" velocity = "${velocity}"/>
@@ -242,5 +281,5 @@
         <dynamics damping="0.205" friction="0.15"/>
 	</joint>
-	<joint name="joint3" type="revolute">
+	<joint name="link2_to_link3" type="revolute">
 		<axis xyz=" 0 0 1"/>
 		<limit effort = "${effort}" lower = "-2.879793" upper = "2.879793" velocity = "${velocity}"/>
@@ -250,5 +289,5 @@
         <dynamics damping="0.21" friction="0.41"/>
 	</joint>
-	<joint name="joint4" type="revolute">
+	<joint name="link3_to_link4" type="revolute">
 		<axis xyz=" 0 0 1"/>
 		<limit effort = "${effort}" lower = "-2.879793" upper = "2.879793" velocity = "${velocity}"/>
@@ -258,5 +297,5 @@
         <dynamics damping="0.10" friction="0.20"/>
 	</joint>
-	<joint name="joint5" type="revolute">
+	<joint name="link4_to_link5" type="revolute">
 		<axis xyz=" 0 0 1"/>
 		<limit effort = "${effort}" lower = "-2.879793" upper = "2.879793" velocity = "${velocity}"/>
@@ -266,5 +305,5 @@
         <dynamics damping="0.01" friction="0.005"/>
 	</joint>
-	<joint name="joint6" type="revolute">
+	<joint name="link5_to_link5_flange" type="revolute">
 		<axis xyz=" 0 0 1"/>
 		<limit effort = "${effort}" lower = "-3.05" upper = "3.05" velocity = "${velocity}"/>
@@ -284,3 +323,9 @@
   <child link="spectrometer"/>
 </joint>
+    <xacro:default_transmission joint_name="base_link_to_link1"/>
+    <xacro:default_transmission joint_name="link1_to_link2"/>
+    <xacro:default_transmission joint_name="link2_to_link3"/>
+    <xacro:default_transmission joint_name="link3_to_link4"/>
+    <xacro:default_transmission joint_name="link4_to_link5"/>
+    <xacro:default_transmission joint_name="link5_to_link5_flange"/>
 </robot>

File: src/mycobot_ros2/mycobot_gazebo/urdf/ros2_control/classic_gazebo/mycobot_280.urdf.xacro (robot description, xacro)
@@ -32,5 +32,5 @@
 	<xacro:property name="velocity" value="2.792527"/>
 	<!-- ********** LINKS ********** -->
-  <link name="joint1">
+  <link name="base_link">
     <visual>
       <geometry>
@@ -236,5 +236,5 @@
   </collision>
 </link>
-  <gazebo reference="joint1">
+  <gazebo reference="base_link">
         <material>Gazebo/Green</material>
     </gazebo>
@@ -262,16 +262,16 @@
 	<joint name="virtual_joint" type="fixed">
 		<parent link="world"/>
-		<child link="joint1"/>
+		<child link="base_link"/>
 		<origin xyz= "0 0 -0.05" rpy = "0 0 0"/>
 	</joint>
-<joint name="joint1" type="revolute">
+<joint name="base_link_to_link1" type="revolute">
 		<axis xyz="0 0 1"/>
 		<limit effort = "${effort}" lower = "-2.879793" upper = "2.879793" velocity = "${velocity}"/>
-		<parent link="joint1"/>
+		<parent link="base_link"/>
 		<child link="link1"/>
 	    <origin xyz= "0 0 0.13156" rpy = "0 0 ${pi/2}"/>
         <dynamics damping="0.05" friction="0.05"/>
 	</joint>
-	<joint name="joint2" type="revolute">
+	<joint name="link1_to_link2" type="revolute">
 		<axis xyz="0 0 1"/>
 		<limit effort = "${effort}" lower = "-2.879793" upper = "2.879793" velocity = "${velocity}"/>
@@ -281,5 +281,5 @@
         <dynamics damping="0.205" friction="0.15"/>
 	</joint>
-	<joint name="joint3" type="revolute">
+	<joint name="link2_to_link3" type="revolute">
 		<axis xyz=" 0 0 1"/>
 		<limit effort = "${effort}" lower = "-2.879793" upper = "2.879793" velocity = "${velocity}"/>
@@ -289,5 +289,5 @@
         <dynamics damping="0.21" friction="0.41"/>
 	</joint>
-	<joint name="joint4" type="revolute">
+	<joint name="link3_to_link4" type="revolute">
 		<axis xyz=" 0 0 1"/>
 		<limit effort = "${effort}" lower = "-2.879793" upper = "2.879793" velocity = "${velocity}"/>
@@ -297,5 +297,5 @@
         <dynamics damping="0.10" friction="0.20"/>
 	</joint>
-	<joint name="joint5" type="revolute">
+	<joint name="link4_to_link5" type="revolute">
 		<axis xyz=" 0 0 1"/>
 		<limit effort = "${effort}" lower = "-2.879793" upper = "2.879793" velocity = "${velocity}"/>
@@ -305,5 +305,5 @@
         <dynamics damping="0.01" friction="0.005"/>
 	</joint>
-	<joint name="joint6" type="revolute">
+	<joint name="link5_to_link5_flange" type="revolute">
 		<axis xyz=" 0 0 1"/>
 		<limit effort = "${effort}" lower = "-3.05" upper = "3.05" velocity = "${velocity}"/>
@@ -323,9 +323,9 @@
   <child link="spectrometer"/>
 </joint>
-    <xacro:default_transmission joint_name="joint1"/>
-    <xacro:default_transmission joint_name="joint2"/>
-    <xacro:default_transmission joint_name="joint3"/>
-    <xacro:default_transmission joint_name="joint4"/>
-    <xacro:default_transmission joint_name="joint5"/>
-    <xacro:default_transmission joint_name="joint6"/>
+    <xacro:default_transmission joint_name="base_link_to_link1"/>
+    <xacro:default_transmission joint_name="link1_to_link2"/>
+    <xacro:default_transmission joint_name="link2_to_link3"/>
+    <xacro:default_transmission joint_name="link3_to_link4"/>
+    <xacro:default_transmission joint_name="link4_to_link5"/>
+    <xacro:default_transmission joint_name="link5_to_link5_flange"/>
 </robot>

File: src/mycobot_ros2/mycobot_gazebo/urdf/ros2_control/classic_gazebo/mycobot_280_ros2_control.xacro (robot description, xacro)
@@ -1,10 +1,10 @@
 <?xml version="1.0" ?>
 <robot xmlns:xacro="http://wiki.ros.org/xacro" name="mycobot_280">
-    <!-- Interface the robot's hardware with the ROS 2 Control library
-    <ros2_control name="GazeboSystem" type="system">
+    <!-- Interface the robot's hardware with the ROS 2 Control library -->
+    <ros2_control name="RobotSystem" type="system">
         <hardware>
             <plugin>gazebo_ros2_control/GazeboSystem</plugin>
         </hardware>
-        <joint name="joint1">
+        <joint name="base_link_to_link1">
             <command_interface name="position">
                 <param name="min">-2.879793</param>
@@ -13,5 +13,5 @@
             <state_interface name="position"/>
         </joint>
-        <joint name="joint2">
+        <joint name="link1_to_link2">
             <command_interface name="position">
                 <param name="min">-2.879793</param>
@@ -20,5 +20,5 @@
             <state_interface name="position"/>
         </joint>
-        <joint name="joint3">
+        <joint name="link2_to_link3">
             <command_interface name="position">
                 <param name="min">-2.879793</param>
@@ -27,5 +27,5 @@
             <state_interface name="position"/>
         </joint>
-        <joint name="joint4">
+        <joint name="link3_to_link4">
             <command_interface name="position">
                 <param name="min">-2.879793</param>
@@ -34,5 +34,5 @@
             <state_interface name="position"/>
         </joint>
-        <joint name="joint5">
+        <joint name="link4_to_link5">
             <command_interface name="position">
                 <param name="min">-2.879793</param>
@@ -41,54 +41,5 @@
             <state_interface name="position"/>
         </joint>
-        <joint name="joint6">
-            <command_interface name="position">
-                <param name="min">-3.05</param>
-                <param name="max">3.05</param>
-            </command_interface>
-            <state_interface name="position"/>
-        </joint>
-    </ros2_control>
-    -->
-    <!-- Interface the robot's hardware with the ROS 2 Control library -->
-    <ros2_control name="RealRobot" type="system">
-      <hardware>
-          <plugin>mycobot_hardware_interface/MyCobotHardwareInterface</plugin>
-      </hardware>
-        <joint name="joint1">
-            <command_interface name="position">
-                <param name="min">-2.879793</param>
-                <param name="max">2.879793</param>
-            </command_interface>
-            <state_interface name="position"/>
-        </joint>
-        <joint name="joint2">
-            <command_interface name="position">
-                <param name="min">-2.879793</param>
-                <param name="max">2.879793</param>
-            </command_interface>
-            <state_interface name="position"/>
-        </joint>
-        <joint name="joint3">
-            <command_interface name="position">
-                <param name="min">-2.879793</param>
-                <param name="max">2.879793</param>
-            </command_interface>
-            <state_interface name="position"/>
-        </joint>
-        <joint name="joint4">
-            <command_interface name="position">
-                <param name="min">-2.879793</param>
-                <param name="max">2.879793</param>
-            </command_interface>
-            <state_interface name="position"/>
-        </joint>
-        <joint name="joint5">
-            <command_interface name="position">
-                <param name="min">-2.879793</param>
-                <param name="max">2.879793</param>
-            </command_interface>
-            <state_interface name="position"/>
-        </joint>
-        <joint name="joint6">
+        <joint name="link5_to_link5_flange">
             <command_interface name="position">
                 <param name="min">-3.05</param>

File: src/mycobot_ros2/mycobot_moveit_config/config/mycobot_280.ros2_control.xacro (robot description, xacro)
@@ -8,43 +8,43 @@
                 <plugin>mock_components/GenericSystem</plugin>
             </hardware>
-            <joint name="joint1">
+            <joint name="base_link_to_link1">
                 <command_interface name="position"/>
                 <state_interface name="position">
-                  <param name="initial_value">${initial_positions['joint1']}</param>
+                  <param name="initial_value">${initial_positions['base_link_to_link1']}</param>
                 </state_interface>
                 <state_interface name="velocity"/>
             </joint>
-            <joint name="joint2">
+            <joint name="link1_to_link2">
                 <command_interface name="position"/>
                 <state_interface name="position">
-                  <param name="initial_value">${initial_positions['joint2']}</param>
+                  <param name="initial_value">${initial_positions['link1_to_link2']}</param>
                 </state_interface>
                 <state_interface name="velocity"/>
             </joint>
-            <joint name="joint3">
+            <joint name="link2_to_link3">
                 <command_interface name="position"/>
                 <state_interface name="position">
-                  <param name="initial_value">${initial_positions['joint3']}</param>
+                  <param name="initial_value">${initial_positions['link2_to_link3']}</param>
                 </state_interface>
                 <state_interface name="velocity"/>
             </joint>
-            <joint name="joint4">
+            <joint name="link3_to_link4">
                 <command_interface name="position"/>
                 <state_interface name="position">
-                  <param name="initial_value">${initial_positions['joint4']}</param>
+                  <param name="initial_value">${initial_positions['link3_to_link4']}</param>
                 </state_interface>
                 <state_interface name="velocity"/>
             </joint>
-            <joint name="joint5">
+            <joint name="link4_to_link5">
                 <command_interface name="position"/>
                 <state_interface name="position">
-                  <param name="initial_value">${initial_positions['joint5']}</param>
+                  <param name="initial_value">${initial_positions['link4_to_link5']}</param>
                 </state_interface>
                 <state_interface name="velocity"/>
             </joint>
-            <joint name="joint6">
+            <joint name="link5_to_link5_flange">
                 <command_interface name="position"/>
                 <state_interface name="position">
-                  <param name="initial_value">${initial_positions['joint6']}</param>
+                  <param name="initial_value">${initial_positions['link5_to_link5_flange']}</param>
                 </state_interface>
                 <state_interface name="velocity"/>

Commit message: Robot working with given poses code now

File: src/mycobot_ros2/mycobot_description/urdf/mycobot_280_urdf.xacro (robot description, xacro)
@@ -1,25 +1,5 @@
-<?xml version="1.0" ?>
-<robot xmlns:xacro="http://wiki.ros.org/xacro" name="mycobot_280">
-    <xacro:include filename="$(find mycobot_gazebo)/urdf/ros2_control/classic_gazebo/mycobot_280_classic_gazebo.xacro"/>
-    <xacro:include filename="$(find mycobot_gazebo)/urdf/ros2_control/classic_gazebo/mycobot_280_ros2_control.xacro"/>
-    <xacro:macro name="default_transmission" params="joint_name">
-        <transmission name="transmission_${joint_name}">
-            <plugin>transmission_interface/SimpleTransmission</plugin>
-            <actuator name="actuator_${joint_name}" role="actuator_${joint_name}"/>
-            <joint name="${joint_name}" role="${joint_name}">
-                <mechanical_reduction>1.0</mechanical_reduction>
-            </joint>
-        </transmission>
-    </xacro:macro>
+<?xml version="1.0"?>
+<robot  xmlns:xacro="http://www.ros.org/wiki/xacro" name="firefighter" >
 <xacro:property name="width" value=".2" />
-  <material name="white">
-        <color rgba="1 1 1 1"/>
-    </material>
-    <material name="orange">
-        <color rgba="1 0.3 0.1 1"/>
-    </material>
-    <material name="blue">
-        <color rgba="0.2 0.2 1 1"/>
-    </material>
 <material name="silver">
   <color rgba="0.75 0.75 0.75 1.0"/>
@@ -32,5 +12,5 @@
 	<xacro:property name="velocity" value="2.792527"/>
 	<!-- ********** LINKS ********** -->
-  <link name="base_link">
+  <link name="joint1">
     <visual>
       <geometry>
@@ -196,5 +176,5 @@
 		</inertial>
   </link>
-    <link name="holder">
+  <link name="holder">
   <inertial>
     <origin xyz="9.542063908505497e-10 4.713475046347886e-13 0.051986133375594434" rpy="0 0 0"/>
@@ -236,25 +216,4 @@
   </collision>
 </link>
-  <gazebo reference="base_link">
-        <material>Gazebo/Green</material>
-    </gazebo>
-    <gazebo reference="link1">
-        <material>Gazebo/Blue</material>
-    </gazebo>
-    <gazebo reference="link2">
-        <material>Gazebo/Orange</material>
-    </gazebo>
-<gazebo reference="link3">
-        <material>Gazebo/Green</material>
-    </gazebo>
-    <gazebo reference="link4">
-        <material>Gazebo/Blue</material>
-    </gazebo>
-    <gazebo reference="link5">
-        <material>Gazebo/Orange</material>
-    </gazebo>
-      <gazebo reference="link5_flange">
-        <material>Gazebo/Green</material>
-    </gazebo>
 <!-- ********** JOINTS ********** -->
 <!-- Attach the robot base to the world frame with no initial offset or rotation. -->
@@ -262,16 +221,18 @@
 	<joint name="virtual_joint" type="fixed">
 		<parent link="world"/>
-		<child link="base_link"/>
-		<origin xyz= "0 0 -0.05" rpy = "0 0 0"/>
-	</joint>
-<joint name="base_link_to_link1" type="revolute">
+		<child link="joint1"/>
+		<origin xyz= "0 0 0" rpy = "0 0 0"/>
+	</joint>
+	<!-- Define the joint name and its type as "fixed". A fixed joint
+	means the two connected links cannot move relative to each other. -->
+		<joint name="joint1" type="revolute">
 		<axis xyz="0 0 1"/>
 		<limit effort = "${effort}" lower = "-2.879793" upper = "2.879793" velocity = "${velocity}"/>
-		<parent link="base_link"/>
+		<parent link="joint1"/>
 		<child link="link1"/>
 	    <origin xyz= "0 0 0.13156" rpy = "0 0 ${pi/2}"/>
         <dynamics damping="0.05" friction="0.05"/>
 	</joint>
-	<joint name="link1_to_link2" type="revolute">
+	<joint name="joint2" type="revolute">
 		<axis xyz="0 0 1"/>
 		<limit effort = "${effort}" lower = "-2.879793" upper = "2.879793" velocity = "${velocity}"/>
@@ -281,5 +242,5 @@
         <dynamics damping="0.205" friction="0.15"/>
 	</joint>
-	<joint name="link2_to_link3" type="revolute">
+	<joint name="joint3" type="revolute">
 		<axis xyz=" 0 0 1"/>
 		<limit effort = "${effort}" lower = "-2.879793" upper = "2.879793" velocity = "${velocity}"/>
@@ -289,5 +250,5 @@
         <dynamics damping="0.21" friction="0.41"/>
 	</joint>
-	<joint name="link3_to_link4" type="revolute">
+	<joint name="joint4" type="revolute">
 		<axis xyz=" 0 0 1"/>
 		<limit effort = "${effort}" lower = "-2.879793" upper = "2.879793" velocity = "${velocity}"/>
@@ -297,5 +258,5 @@
         <dynamics damping="0.10" friction="0.20"/>
 	</joint>
-	<joint name="link4_to_link5" type="revolute">
+	<joint name="joint5" type="revolute">
 		<axis xyz=" 0 0 1"/>
 		<limit effort = "${effort}" lower = "-2.879793" upper = "2.879793" velocity = "${velocity}"/>
@@ -305,5 +266,5 @@
         <dynamics damping="0.01" friction="0.005"/>
 	</joint>
-	<joint name="link5_to_link5_flange" type="revolute">
+	<joint name="joint6" type="revolute">
 		<axis xyz=" 0 0 1"/>
 		<limit effort = "${effort}" lower = "-3.05" upper = "3.05" velocity = "${velocity}"/>
@@ -323,9 +284,3 @@
   <child link="spectrometer"/>
 </joint>
-    <xacro:default_transmission joint_name="base_link_to_link1"/>
-    <xacro:default_transmission joint_name="link1_to_link2"/>
-    <xacro:default_transmission joint_name="link2_to_link3"/>
-    <xacro:default_transmission joint_name="link3_to_link4"/>
-    <xacro:default_transmission joint_name="link4_to_link5"/>
-    <xacro:default_transmission joint_name="link5_to_link5_flange"/>
 </robot>
