Commit message: fully working

File: src/mycobot-ros2-fix/mycobot_280_description/config/mycobot_280.ros2_control.xacro (robot description, xacro)
@@ -85,6 +85,6 @@
       <joint name="${prefix}joint6">
         <command_interface name="position">
-          <param name="min">${joint6_lower_limit}</param>
-          <param name="max">${joint6_upper_limit}</param>
+          <param name="min">0</param>
+          <param name="max">0</param>
         </command_interface>
         <state_interface name="position">

File: src/mycobot-ros2-fix/mycobot_280_description/config/mycobot_280_macro.xacro (robot description, xacro)
@@ -240,5 +240,5 @@
       <origin xyz="${joint6_x} ${joint6_y} ${joint6_z}" rpy="${joint6_roll} ${joint6_pitch} ${joint6_yaw}" />
       <axis xyz="0 0 1" />
-      <limit lower="${joint6_lower_limit}" upper="${joint6_upper_limit}"
+      <limit lower="0" upper="0"
              effort="${joint6_effort_limit}" velocity="${joint6_velocity_limit}"/>
       <dynamics damping="0" friction="0"/>

File: src/mycobot-ros2-fix/mycobot_280_description/config/mycobot_urdf.urdf (robot description, URDF)
Before this commit: robot mycobot_280, 9 links, 8 joints
Joints:
- joint joint6: limit lower=-3.14 upper=3.14159 effort=1000.0 velocity=0 -> lower=0 upper=0 effort=1000.0 velocity=0
